File: Eagle files/EEZ DIB PREL6 r1B1.sch (EAGLE design)
At the start: 65 parts, among them IC1 STM32F030C6T6, IC2 74HC1G126DBVT, IC3 M24C32-WMN6P, IC4 LP2985-33DBVR, K1 RT424005, K2 RT424005, K3 RT424005, K4 RT424005, K5 RT424005, K6 RT424005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

Commit message: BOM added, improved PCB clearances
Parts:
- C8: device rcl:C-EUC0805 -> rcl:C-EUC1206
Other:
- note added: "2 x 16-pin front panel connector"
- note added: "K1-COMM"
- note added: "K1-NO"
- note added: "K2-COMM"
- note added: "K2-NC"
- note added: "K2-NO"
- note added: "K3-COMM"
- note added: "K3-NC"
- note added: "K3-NO"
- note added: "K4-COMM"
- note added: "K4-NC"
- note added: "K4-NO"
- note added: "K5-COMM"
- note added: "K5-NC"
- note added: "K5-NO"
- note added: "K6-COMM"
- note added: "K6-NO"

Commit message: UART relocated
Connections:
- removed net OUT22: IC1.PC13
- removed net OUT23: IC1.PC14-OSC32_IN
- net UART_RX: now also IC1.PA10; no longer IC1.PA15
Changed lines of the file:
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@@
-</segment>
-</net>
-<net name="OUT22" class="0">
-<segment>
-<wire x1="170.18" y1="114.3" x2="182.88" y2="114.3" width="0.1524" layer="91"/>
-<label x="170.18" y="114.935" size="1.27" layer="102"/>
-<pinref part="IC1" gate="G$1" pin="PC13"/>
-</segment>
-</net>
-<net name="OUT23" class="0">
-<segment>
-<pinref part="IC1" gate="G$1" pin="PC14-OSC32_IN"/>
-<wire x1="182.88" y1="111.76" x2="170.18" y2="111.76" width="0.1524" layer="91"/>
-<label x="170.18" y="112.395" size="1.27" layer="102"/>
 </segment>
 </net>
@@
 <net name="UART_RX" class="0">
 <segment>
-<pinref part="IC1" gate="G$1" pin="PA15"/>
-<wire x1="223.52" y1="129.54" x2="223.52" y2="142.24" width="0.1524" layer="91"/>
-<label x="222.885" y="132.08" size="1.27" layer="102" rot="R90"/>
-</segment>
-<segment>
+<label x="243.84" y="104.775" size="1.27" layer="102"/>
+<pinref part="IC1" gate="G$1" pin="PA10"/>
+<wire x1="241.3" y1="104.14" x2="251.46" y2="104.14" width="0.1524" layer="91"/>
+</segment>
+<segment>

Commit message: debug connector update
Parts:
- X1: value N.C. -> SSW-106-02-S-S; device EEZ_connectors:22-23-2061 -> con-samtec:SSW-106-02-S-S
Connections:
- net GND: now also X1-3.1; no longer X1-3.S
- net SWCLK: now also X1-2.1; no longer X1-2.S
- net SWDIO: now also X1-4.1; no longer X1-4.S
Changed lines of the file:
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@@
 <part name="IC2" library="EEZ_TI" deviceset="74HC1G126" device="DBVT"/>
 <part name="SUPPLY51" library="supply2" deviceset="GND" device=""/>
-<part name="X1" library="EEZ_connectors" deviceset="22-23-2061" device="" value="N.C."/>
 <part name="FM2" library="EEZ_Lib1" deviceset="FIDUCIAL" device="_2"/>
 <part name="FM1" library="EEZ_Lib1" deviceset="FIDUCIAL" device="_2"/>
@@
 <part name="R6" library="rcl" deviceset="R-EU_" device="R0805" value="100K"/>
 <part name="R7" library="rcl" deviceset="R-EU_" device="R0805" value="100K"/>
+<part name="X1" library="con-samtec" deviceset="SSW-106-02-S-S" device=""/>
 </parts>
 <sheets>
@@
 <attribute name="VALUE" x="168.275" y="159.385" size="1.778" layer="96" rot="MR0"/>
 </instance>
-<instance part="X1" gate="-2" x="175.26" y="167.64" smashed="yes">
-<attribute name="NAME" x="177.8" y="166.878" size="1.524" layer="95"/>
-</instance>
-<instance part="X1" gate="-3" x="175.26" y="162.56" smashed="yes">
-<attribute name="NAME" x="177.8" y="161.798" size="1.524" layer="95"/>
-</instance>
-<instance part="X1" gate="-4" x="175.26" y="165.1" smashed="yes">
-<attribute name="NAME" x="177.8" y="164.338" size="1.524" layer="95"/>
-</instance>
 <instance part="RN1" gate="-4" x="22.86" y="147.32" smashed="yes">
 <attribute name="NAME" x="26.035" y="147.447" size="1.27" layer="95"/>
@@
 <instance part="FM2" gate="FD" x="137.16" y="5.08" smashed="yes"/>
 <instance part="FM1" gate="FD" x="129.54" y="5.08" smashed="yes"/>
+<instance part="X1" gate="-2" x="177.8" y="167.64" smashed="yes" rot="MR0">
+<attribute name="NAME" x="180.848" y="168.402" size="1.524" layer="95" rot="MR180"/>
+</instance>
+<instance part="X1" gate="-3" x="177.8" y="162.56" smashed="yes" rot="MR0">
+<attribute name="NAME" x="180.848" y="163.322" size="1.524" layer="95" rot="MR180"/>
+</instance>
+<instance part="X1" gate="-4" x="177.8" y="165.1" smashed="yes" rot="MR0">
+<attribute name="NAME" x="180.848" y="165.862" size="1.524" layer="95" rot="MR180"/>
+</instance>
 </instances>
 <busses>
@@
 </segment>
 <segment>
-<pinref part="X1" gate="-3" pin="S"/>
-<wire x1="172.72" y1="162.56" x2="170.18" y2="162.56" width="0.1524" layer="91"/>
 <pinref part="SUPPLY51" gate="GND" pin="GND"/>
+<pinref part="X1" gate="-3" pin="1"/>
+<wire x1="175.26" y1="162.56" x2="170.18" y2="162.56" width="0.1524" layer="91"/>
 </segment>
 </net>
@@
 </segment>
 <segment>
-<wire x1="152.4" y1="165.1" x2="172.72" y2="165.1" width="0.1524" layer="91"/>
+<wire x1="152.4" y1="165.1" x2="175.26" y2="165.1" width="0.1524" layer="91"/>
 <label x="152.4" y="165.735" size="1.27" layer="102"/>
-<pinref part="X1" gate="-4" pin="S"/>
+<pinref part="X1" gate="-4" pin="1"/>
 </segment>
 </net>
@@
 </segment>
 <segment>
-<wire x1="152.4" y1="167.64" x2="172.72" y2="167.64" width="0.1524" layer="91"/>
+<wire x1="152.4" y1="167.64" x2="175.26" y2="167.64" width="0.1524" layer="91"/>
 <label x="152.4" y="168.275" size="1.27" layer="102"/>
-<pinref part="X1" gate="-2" pin="S"/>
-</segment>
-</net>
+<pinref part="X1" gate="-2" pin="1"/>
+</segment>
+</net>

Commit message: IC2 package update
Parts:
- IC2: value 74HC1G126DBVT -> 74HC1G126GW,125; device EEZ_TI:74HC1G126DBVT -> EEZ_Lib1:74HC1G126GW,125
Changed lines of the file:
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@@
 <part name="SUPPLY47" library="supply2" deviceset="GND" device=""/>
 <part name="+3V7" library="supply1" deviceset="+3V3" device=""/>
-<part name="IC2" library="EEZ_TI" deviceset="74HC1G126" device="DBVT"/>
+<part name="IC2" library="EEZ_Lib1" deviceset="74HC1G126" device="GW,125"/>
 <part name="SUPPLY51" library="supply2" deviceset="GND" device=""/>
 <part name="FM2" library="EEZ_Lib1" deviceset="FIDUCIAL" device="_2"/>
