File: EDA files/EEZ DIB PREL6 r1B1.brd (EAGLE design)
At the start: 146 x 95 mm, 66 parts, among them IC1 STM32F030C6T6, IC2 74HC1G126GW,125, IC3 M24C32-WMN6P, IC4 LP2985-33DBVR, K1 RT424005, K2 RT424005, K3 RT424005, K4 RT424005, K5 RT424005, K6 RT424005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

Commit message: front panel connectors position adjusted
Parts:
- moved X3 0.30 mm to (12.0, 65.0)
- moved X4 0.30 mm to (12.0, 33.0)
