File: EDA files/EEZ DIB PREL6 r1B4.brd (EAGLE design)
At the start: 146 x 95 mm, 68 parts, among them IC1 STM32F030C6T6, IC2 74HC1G126GW,125, IC3 M24C32-WMN6P, IC4 LP2985-33DBVR, K1 RT424005, K2 RT424005, K3 RT424005, K4 RT424005, K5 RT424005, K6 RT424005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

Commit message: #4, OSHW UID
Parts:
- removed ZD2, ZD3, ZD4, ZD5, ZD6: MM3Z18VT1G, EEZ_Lib1:SOD323-R
- added FM3: FIDUCIAL_2, EEZ_Lib1:FIDUCIAL_DUAL
- added U$3: HR000005, OSHWA:CERT-SMALL-SILK
- moved ZD1 71.1 mm to (132.3, 64.4), turned to 180 degrees
- moved D4 7.94 mm to (63.5, 50.8), turned to 270 degrees
- moved D5 7.94 mm to (99.1, 50.8), turned to 270 degrees
- moved D6 7.94 mm to (134.9, 50.8), turned to 270 degrees
- moved FM1 1.12 mm to (15.0, 92.5)
Connections:
- removed net N$10: D5.A, ZD5.A
- removed net N$6: D3.A, ZD3.A
- removed net N$8: D4.A, ZD4.A
- removed net N$9: K4.A1, Q4.3, ZD4.C
- removed net N$98: D6.A, ZD6.A
- net +5V: now also ZD1.A; no longer D1.C, D2.C, D3.C, D4.C, D5.C, D6.C
- net N$1: now also D4.A, K4.A1, Q4.3; no longer D1.A, ZD1.A
- net N$100: now also D6.A; no longer ZD6.C
- net N$11: now also D5.A; no longer ZD5.C
- net N$2: now also D1.A; no longer ZD1.C
- net N$3: now also D1.C, D2.C, D3.C, D4.C, D5.C, D6.C, ZD1.C; no longer D2.A, ZD2.A
- net N$4: now also D2.A; no longer ZD2.C
- net N$7: now also D3.A; no longer ZD3.C
Routing:
- net N$3: track 1.84 -> 155.4 mm, vias 0 -> 10
- net N$9: track 51.8 -> 0.00 mm, vias 1 -> 0
- net N$1: track 1.84 -> 52.7 mm, vias 0 -> 1
- net +5V: track 364.4 -> 341.6 mm, vias 2 -> 3
- net N$2: track 8.93 -> 11.1 mm
- net N$4: track 8.93 -> 11.1 mm
- net N$7: track 9.14 -> 11.1 mm
- net N$98: track 1.91 -> 0.00 mm
- net N$8: track 1.91 -> 0.00 mm
- net N$10: track 1.91 -> 0.00 mm
- net N$6: track 1.84 -> 0.00 mm
Other:
- board text added: "+VAUX 2 NRESET 4 SYNC 6 SSDA 8 IRQ 10 CSB 12 MISO 14 GND 16 A2 18 GND 20 +12V 22 +5V 24 BOOT 26 UART_TX 28"
- board text added: "1 +3V3 3 NFAULT 5 SSCL 7 GND 9 CSA 11 GND 13 SCLK 15 MOSI 17 A0 19 A1 21 +12V 23 +5V 25 GND 27 UART_RX"
- board text added: "DIB (bottom view)"
- board text added: "EEZ DIB PREL6 (12/2020 r1B3)"
- board text added: "EEZ DIB PREL6 (12/2020 r1B3) Project source code: github.com/eez-open"
- board text removed: "EEZ DIB PREL6 (09/2020 r1B3)"
- board text removed: "EEZ DIB PREL6 (09/2020 r1B3) Project source code: github.com/eez-open"

Commit message: PCB ID added
Connections:
- new net N$6: IC1.6
- net GND: now also IC1.5
Routing:
- net GND: track 254.0 -> 255.5 mm, vias 30 -> 31
Other:
- board text added: "EEZ DIB PREL6 (01/2021 r1B4)"
- board text added: "EEZ DIB PREL6 (01/2021 r1B4) Project source code: github.com/eez-open"
- board text removed: "EEZ DIB PREL6 (12/2020 r1B3)"
- board text removed: "EEZ DIB PREL6 (12/2020 r1B3) Project source code: github.com/eez-open"
Changed lines of the file:
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@@
 <layer number="56" name="wert" color="7" fill="1" visible="no" active="no"/>
 <layer number="57" name="tCAD" color="7" fill="1" visible="no" active="no"/>
+<layer number="88" name="SimResults" color="9" fill="1" visible="no" active="yes"/>
+<layer number="89" name="SimProbes" color="9" fill="1" visible="no" active="yes"/>
 <layer number="90" name="Modules" color="7" fill="1" visible="no" active="no"/>
 <layer number="91" name="Nets" color="2" fill="1" visible="no" active="no"/>
@@
 <layer number="111" name="111" color="7" fill="1" visible="no" active="no"/>
 <layer number="112" name="tSilk" color="7" fill="1" visible="no" active="no"/>
+<layer number="113" name="ReferenceLS" color="7" fill="1" visible="no" active="yes"/>
 <layer number="114" name="Änderung" color="7" fill="1" visible="no" active="no"/>
+<layer number="115" name="CH1" color="13" fill="1" visible="no" active="yes"/>
 <layer number="116" name="Patch_BOT" color="7" fill="1" visible="no" active="no"/>
+<layer number="117" name="CH2" color="9" fill="1" visible="no" active="yes"/>
 <layer number="118" name="Rect_Pads" color="7" fill="1" visible="no" active="no"/>
+<layer number="119" name="CH3" color="12" fill="1" visible="no" active="yes"/>
 <layer number="120" name="lotbs" color="7" fill="1" visible="no" active="no"/>
 <layer number="121" name="_tsilk" color="7" fill="1" visible="no" active="no"/>
@@
 <layer number="127" name="_tValues" color="7" fill="1" visible="no" active="no"/>
 <layer number="128" name="_bValues" color="7" fill="1" visible="no" active="no"/>
+<layer number="129" name="sram_cmd" color="13" fill="1" visible="no" active="yes"/>
+<layer number="130" name="sram_ctrl" color="2" fill="1" visible="no" active="yes"/>
 <layer number="131" name="tAdjust" color="7" fill="1" visible="no" active="no"/>
 <layer number="132" name="bAdjust" color="7" fill="1" visible="no" active="no"/>
+<layer number="133" name="corrections" color="12" fill="1" visible="no" active="yes"/>
 <layer number="144" name="Drill_legend" color="7" fill="1" visible="no" active="no"/>
 <layer number="148" name="Document_mirrored" color="7" fill="1" visible="no" active="no"/>
@@
 <dimension x1="-10" y1="81" x2="-11" y2="17" x3="-12" y3="49" textsize="2" layer="47" dtype="vertical"/>
 <text x="23.1675" y="3.2345" size="1.27" layer="21" font="vector" ratio="10" rot="SR0">EEZ DIB PREL6
-(12/2020 r1B3)</text>
-<text x="140.5215" y="48.861" size="1.27" layer="22" font="vector" ratio="10" rot="SMR90">EEZ DIB PREL6 (12/2020 r1B3)
+(01/2021 r1B4)</text>
+<text x="140.5215" y="48.861" size="1.27" layer="22" font="vector" ratio="10" rot="SMR90">EEZ DIB PREL6 (01/2021 r1B4)
 Project source code: github.com/eez-open</text>
 <rectangle x1="17.145" y1="7.62" x2="39.243" y2="13.2715" layer="21"/>
@@
 <element name="IC2" library="EEZ_Lib1" package="SOT65P210X110-5N" value="74HC1G126GW,125" x="101.5365" y="18.288" smashed="yes">
 <attribute name="NAME" x="100.3141" y="19.558" size="1.016" layer="25" ratio="10" rot="SR0"/>
-<attribute name="VALUE" x="96.3676" y="17.907" size="0.6096" layer="27" ratio="10" rot="SR0"/>
+<attribute name="VALUE" x="96.8121" y="17.3355" size="0.6096" layer="27" ratio="10" rot="SR0"/>
 </element>
 <element name="EEZ_SIGNATURE" library="EEZ_Lib1" package="SIGNATURE_5MM" value="SIGNATURESMALL" x="19.8585" y="4.6765" smashed="yes" rot="R180"/>
@@
 <wire x1="135.0645" y1="25.8445" x2="135.0645" y2="27.1145" width="0.3048" layer="1"/>
 <contactref element="GND" pad="1"/>
+<contactref element="IC1" pad="5"/>
+<via x="120.396" y="16.891" extent="1-16" drill="0.4" shape="octagon"/>
+<wire x1="118.9101" y1="16.891" x2="120.396" y2="16.891" width="0.2032" layer="1"/>
 </signal>
 <signal name="DIB_A0">
@@
 <wire x1="66.8955" y1="80.2005" x2="66.6265" y2="79.9315" width="0.4064" layer="16"/>
 </signal>
+<signal name="N$6">
+<contactref element="IC1" pad="6"/>
+</signal>
 </signals>
